File: mobile-sensor-pcb.sch (KiCad schematic (older format))
At the start: 93 parts, among them J1 SMA, J2 USB_OTG, J3 JST PH, Q1 PNP-BJT-BIASED_SOT, SW1 RESET, SW2 ON/OFF, U1 3M_2908-05WB-MG, U10 LP2980AIM5-3.3/NOPB, U11 LP2980AIM5-3.3/NOPB, U12 LP2980AIM5-3.3/NOPB, U13 TPS61030RSA, U2 74HC4050, U3 FGPMMOPA6H, U4 RT9193, U5 MIC5219, U6 MCP73831T-2ACI/OT, U7 MAX31855KASA, U8 MAX31855KASA, U9 MAX31855KASA, X1 XBEE

Commit message: Fix a few bad connections, start to lay out PCB
Parts:
- C1, C10, C11, C12, C2, C3, C4, C5, C6, C7, C8, C9: value 10 uF -> 10uF
- C14, C15, C16: value 100 nF -> 100nF
- C17, C18, C19: value 10 nF -> 10nF
- C20: value 100 uF -> 100uF
- C21: value 2.2 uF -> 2.2uF
Connections:
- net GND: now also J1.3 (GND2), J1.4 (GND3), J2.6 (shield), U13.6 (PGND), U13.7 (PGND)
- net XBEE-3V3: now also C14.1
- net at FB7.2, U3.1 (VCC): now also C16.1
- net at C20.1, C21.1, F1.2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: now also U13.15 (VOUT)
- net at Q1.1 (B): now also U13.12 (LBO)
- no-connect marks 94 -> 95
Other:
- moved on the sheet: C16, Q1
